File: pdp-backplane.kicad_sch (KiCad schematic)
At the start: 54 parts, among them J1 Power Control, J2 ATX-20, J3 Molex Power, Q1 Bus_QBUS, Q10 Bus_QBUS, Q11 Bus_QBUS, Q12 Bus_QBUS, Q13 Bus_QBUS, Q14 Bus_QBUS, Q15 Bus_QBUS, Q16 Bus_QBUS, Q2 Bus_QBUS, Q3 Bus_QBUS, Q4 Bus_QBUS, Q5 Bus_QBUS, Q6 Bus_QBUS, Q7 Bus_QBUS, Q8 Bus_QBUS, Q9 Bus_QBUS

Commit message: add: new version
Connections:
- net at JP10.2 (B), Q10.AN2 (BIAKO): now also JP12.1 (A), Q12.AM2 (BIAKI); no longer JP24.1 (A), Q11.AM2 (BIAKI)
- net at JP26.1 (A), Q13.AM2 (BIAKI): now also JP24.2 (B), Q11.AN2 (BIAKO); no longer JP12.2 (B), Q12.AN2 (BIAKO)
- net at JP16.1 (A), Q3.AM2 (BIAKI): now also JP4.2 (B), Q4.AN2 (BIAKO); no longer JP2.2 (B), Q2.AN2 (BIAKO)
- net at JP16.2 (B), Q3.AN2 (BIAKO): now also JP18.1 (A), Q5.AM2 (BIAKI); no longer JP4.1 (A), Q4.AM2 (BIAKI)
- net at JP15.1 (A), Q3.AR2 (BDMGI): now also JP3.2 (B), Q4.AS2 (BDMGO); no longer JP1.2 (B), Q2.AS2 (BDMGO)
- net at JP15.2 (B), Q3.AS2 (BDMGO): now also JP17.1 (A), Q5.AR2 (BDMGI); no longer JP3.1 (A), Q4.AR2 (BDMGI)
- net at JP8.1 (A), Q8.AM2 (BIAKI): now also JP6.2 (B), Q6.AN2 (BIAKO); no longer JP20.2 (B), Q7.AN2 (BIAKO)
- net at JP8.2 (B), Q8.AN2 (BIAKO): now also JP20.1 (A), Q7.AM2 (BIAKI); no longer JP22.1 (A), Q9.AM2 (BIAKI)
- net at JP7.1 (A), Q8.AR2 (BDMGI): now also JP5.2 (B), Q6.AS2 (BDMGO); no longer JP19.2 (B), Q7.AS2 (BDMGO)
- net at JP7.2 (B), Q8.AS2 (BDMGO): now also JP19.1 (A), Q7.AR2 (BDMGI); no longer JP21.1 (A), Q9.AR2 (BDMGI)
- net at JP9.2 (B), Q10.AS2 (BDMGO): now also JP11.1 (A), Q12.AR2 (BDMGI); no longer JP23.1 (A), Q11.AR2 (BDMGI)
- net at Q16.AN2 (BIAKO): now also JP28.2 (B), Q15.AR2 (BDMGI)
- net at Q16.AS2 (BDMGO): now also JP27.2 (B), Q15.AM2 (BIAKI)
- net at JP14.2 (B), JP28.1 (A), Q14.AN2 (BIAKO): now also Q16.AM2 (BIAKI); no longer Q15.AM2 (BIAKI)
- net at JP25.1 (A), Q13.AR2 (BDMGI): now also JP23.2 (B), Q11.AS2 (BDMGO); no longer JP11.2 (B), Q12.AS2 (BDMGO)
- net at JP13.2 (B), JP27.1 (A), Q14.AS2 (BDMGO): now also Q16.AR2 (BDMGI); no longer Q15.AR2 (BDMGI)
- new net: JP2.2 (B), JP4.1 (A), Q2.AN2 (BIAKO), Q4.AM2 (BIAKI)
- new net: JP1.2 (B), JP3.1 (A), Q2.AS2 (BDMGO), Q4.AR2 (BDMGI)
- new net: JP12.2 (B), JP24.1 (A), Q11.AM2 (BIAKI), Q12.AN2 (BIAKO)
- new net: JP11.2 (B), JP23.1 (A), Q11.AR2 (BDMGI), Q12.AS2 (BDMGO)
- new net: JP20.2 (B), JP22.1 (A), Q7.AN2 (BIAKO), Q9.AM2 (BIAKI)
- new net: JP19.2 (B), JP21.1 (A), Q7.AS2 (BDMGO), Q9.AR2 (BDMGI)
- now unconnected: Q15.AN2 (BIAKO), Q15.AS2 (BDMGO)
